File: usb.kicad_sch (KiCad schematic)
At the start: 4 parts, among them J1 USB_OTG, U7 ECMF02-2AMX6

Commit message: Finished USB JTAG connectors and cleaned up schematic
Parts:
- removed CR2, CR3: ESDA7P60-1U1M, ZDO_1610_STM, symbol ESDA7P60_1U1M:ESDA7P60-1U1M
- removed J1: USB_OTG, symbol Connector:USB_OTG
- removed U7: ECMF02-2AMX6, Package_DFN_QFN:ST_UQFN-6L_1.5x1.7mm_P0.5mm, symbol Power_Protection:ECMF02-2AMX6
