File: ethernet.kicad_sch (KiCad schematic)
At the start: 50 parts, among them U7 LAN8720A, U8 ARJM11C7-114-BA-EW2, Y1 25MHz

Commit message: Added all footprints and kicked off pcb design
Parts:
- CR9: footprint (none) -> footprints:SOT23-6L_STM
- FB1: footprint (none) -> Inductor_SMD:L_0805_2012Metric
- U8: footprint (none) -> ARJM11C7-114-BA-EW2_ABR
Changed lines of the file:
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@@
 	)
 	(symbol
-		(lib_id "ARJM11C7_114_BA_EW2:ARJM11C7-114-BA-EW2")
-		(at 204.47 119.38 0)
-		(unit 1)
-		(exclude_from_sim no)
-		(in_bom yes)
-		(on_board yes)
-		(dnp no)
-		(fields_autoplaced yes)
-		(property "Reference" "U8"
-			(at 224.79 109.22 0)
-			(effects
-				(font
-					(size 1.524 1.524)
-				)
-			)
-		)
-		(property "Value" "ARJM11C7-114-BA-EW2"
-			(at 224.79 111.76 0)
-			(effects
-				(font
-					(size 1.524 1.524)
-				)
-			)
-		)
-		(property "Footprint" ""
-			(at 241.046 144.526 0)
-			(effects
-				(font
-					(size 1.27 1.27)
-					(italic yes)
-				)
-				(hide yes)
-			)
-		)
-		(property "Datasheet" "ARJM11C7-114-BA-EW2"
-			(at 240.03 141.986 0)
-			(effects
-				(font
-					(size 1.27 1.27)
-					(italic yes)
-				)
-				(hide yes)
-			)
-		)
-		(property "Description" ""
-			(at 204.47 119.38 0)
-			(effects
-				(font
-					(size 1.27 1.27)
-				)
-				(hide yes)
-			)
-		)
-		(pin "12"
-		)
-		(pin "9"
-		)
-		(pin "4"
-		)
-		(pin "10"
-		)
-		(pin "6"
-		)
-		(pin "8"
-		)
-		(pin "2"
-		)
-		(pin "11"
-		)
-		(pin "3"
-		)
-		(pin "13"
-		)
-		(pin "14"
-		)
-		(pin "SH"
-		)
-		(pin "5"
-		)
-		(pin "7"
-		)
-		(pin "1"
-		)
-		(instances
-			(project ""
-				(path "/21bb932a-ec67-4661-9215-0551f718d1c0/df814d64-f889-41f0-8f1a-74d7f134d61e"
-					(reference "U8")
-					(unit 1)
-				)
-			)
-		)
-	)
-	(symbol
 		(lib_id "SparkFun-Capacitor:C")
 		(at 180.34 154.94 0)
@@
 	)
 	(symbol
+		(lib_id "ARJM11C7_114_BA_EW2:ARJM11C7-114-BA-EW2")
+		(at 204.47 119.38 0)
+		(unit 1)
+		(exclude_from_sim no)
+		(in_bom yes)
+		(on_board yes)
+		(dnp no)
+		(fields_autoplaced yes)
+		(property "Reference" "U8"
+			(at 224.79 109.22 0)
+			(effects
+				(font
+					(size 1.524 1.524)
+				)
+			)
+		)
+		(property "Value" "ARJM11C7-114-BA-EW2"
+			(at 224.79 111.76 0)
+			(effects
+				(font
+					(size 1.524 1.524)
+				)
+			)
+		)
+		(property "Footprint" "ARJM11C7-114-BA-EW2_ABR"
+			(at 204.47 119.38 0)
+			(effects
+				(font
+					(size 1.27 1.27)
+					(italic yes)
+				)
+				(hide yes)
+			)
+		)
+		(property "Datasheet" "ARJM11C7-114-BA-EW2"
+			(at 204.47 119.38 0)
+			(effects
+				(font
+					(size 1.27 1.27)
+					(italic yes)
+				)
+				(hide yes)
+			)
+		)
+		(property "Description" ""
+			(at 204.47 119.38 0)
+			(effects
+				(font
+					(size 1.27 1.27)
+				)
+				(hide yes)
+			)
+		)
+		(pin "7"
+		)
+		(pin "12"
+		)
+		(pin "14"
+		)
+		(pin "2"
+		)
+		(pin "6"
+		)
+		(pin "11"
+		)
+		(pin "4"
+		)
+		(pin "10"
+		)
+		(pin "5"
+		)
+		(pin "13"
+		)
+		(pin "1"
+		)
+		(pin "SH"
+		)
+		(pin "8"
+		)
+		(pin "3"
+		)
+		(pin "9"
+		)
+		(instances
+			(project ""
+				(path "/21bb932a-ec67-4661-9215-0551f718d1c0/df814d64-f889-41f0-8f1a-74d7f134d61e"
+					(reference "U8")
+					(unit 1)
+				)
+			)
+		)
+	)
+	(symbol
 		(lib_id "power:GND")
 		(at 144.78 41.91 0)
@@
 			)
 		)
-		(property "Footprint" ""
+		(property "Footprint" "Inductor_SMD:L_0805_2012Metric"
 			(at 92.71 30.988 90)
 			(effects
@@
 			)
 		)
-		(property "Footprint" ""
+		(property "Footprint" "footprints:SOT23-6L_STM"
 			(at 218.44 31.75 0)
 			(effects

Commit message: Layout started
Parts:
- U8: footprint ARJM11C7-114-BA-EW2_ABR -> footprints:ARJM11C7-114-BA-EW2_ABR
- renumbered R104 to R118, R105 to R119, R106 to R120, R107 to R121, R108 to R122, R109 to R123, R110 to R124, R111 to R125, R112 to R126, R113 to R127, R114 to R128, R115 to R129, R116 to R130, R117 to R131, R118 to R132, R119 to R133, R120 to R134, R121 to R135, R122 to R136, R123 to R137, R124 to R138, R125 to R139, R126 to R140, R127 to R141, R128 to R142

Commit message: Component placement
Parts:
- renumbered R118 to R120, R119 to R121, R120 to R122, R121 to R123, R122 to R124, R123 to R125, R124 to R126, R125 to R127, R126 to R128, R127 to R129, R128 to R130, R129 to R131, R130 to R132, R131 to R133, R132 to R134, R133 to R135, R134 to R136, R135 to R137, R136 to R138, R137 to R139, R138 to R140, R139 to R141, R140 to R142, R141 to R143, R142 to R144
Changed lines of the file:
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@@
 		(on_board yes)
 		(dnp no)
-		(property "Reference" "R135"
+		(property "Reference" "R137"
 			(at 63.5 162.5601 90)
 			(effects
@@
 			(project "SBC"
 				(path "/21bb932a-ec67-4661-9215-0551f718d1c0/df814d64-f889-41f0-8f1a-74d7f134d61e"
-					(reference "R135")
+					(reference "R137")
 					(unit 1)
 				)
@@
 		(on_board yes)
 		(dnp no)
-		(property "Reference" "R125"
+		(property "Reference" "R127"
 			(at 48.2599 104.14 90)
 			(effects
@@
 			(project "SBC"
 				(path "/21bb932a-ec67-4661-9215-0551f718d1c0/df814d64-f889-41f0-8f1a-74d7f134d61e"
-					(reference "R125")
+					(reference "R127")
 					(unit 1)
 				)
@@
 		(on_board yes)
 		(dnp no)
-		(property "Reference" "R122"
+		(property "Reference" "R124"
 			(at 234.95 86.3601 90)
 			(effects
@@
 			(project "SBC"
 				(path "/21bb932a-ec67-4661-9215-0551f718d1c0/df814d64-f889-41f0-8f1a-74d7f134d61e"
-					(reference "R122")
+					(reference "R124")
 					(unit 1)
 				)
@@
 		(on_board yes)
 		(dnp yes)
-		(property "Reference" "R142"
+		(property "Reference" "R144"
 			(at 74.93 182.8801 90)
 			(effects
@@
 			(project "SBC"
 				(path "/21bb932a-ec67-4661-9215-0551f718d1c0/df814d64-f889-41f0-8f1a-74d7f134d61e"
-					(reference "R142")
+					(reference "R144")
 					(unit 1)
 				)
@@
 		(on_board yes)
 		(dnp yes)
-		(property "Reference" "R126"
+		(property "Reference" "R128"
 			(at 50.8001 114.3 90)
 			(effects
@@
 			(project "SBC"
 				(path "/21bb932a-ec67-4661-9215-0551f718d1c0/df814d64-f889-41f0-8f1a-74d7f134d61e"
-					(reference "R126")
+					(reference "R128")
 					(unit 1)
 				)
@@
 		(on_board yes)
 		(dnp no)
-		(property "Reference" "R123"
+		(property "Reference" "R125"
 			(at 245.11 86.3601 90)
 			(effects
@@
 			(project "SBC"
 				(path "/21bb932a-ec67-4661-9215-0551f718d1c0/df814d64-f889-41f0-8f1a-74d7f134d61e"
-					(reference "R123")
+					(reference "R125")
 					(unit 1)
 				)
@@
 		(on_board yes)
 		(dnp yes)
-		(property "Reference" "R141"
+		(property "Reference" "R143"
 			(at 63.5 182.8801 90)
 			(effects
@@
 			(project "SBC"
 				(path "/21bb932a-ec67-4661-9215-0551f718d1c0/df814d64-f889-41f0-8f1a-74d7f134d61e"
-					(reference "R141")
+					(reference "R143")
 					(unit 1)
 				)
@@
 		(on_board yes)
 		(dnp no)
-		(property "Reference" "R134"
+		(property "Reference" "R136"
 			(at 52.07 162.5601 90)
 			(effects
@@
 			(project "SBC"
 				(path "/21bb932a-ec67-4661-9215-0551f718d1c0/df814d64-f889-41f0-8f1a-74d7f134d61e"
-					(reference "R134")
+					(reference "R136")
 					(unit 1)
 				)
@@
 		(on_board yes)
 		(dnp no)
-		(property "Reference" "R129"
+		(property "Reference" "R131"
 			(at 153.67 148.5901 90)
 			(effects
@@
 			(project "SBC"
 				(path "/21bb932a-ec67-4661-9215-0551f718d1c0/df814d64-f889-41f0-8f1a-74d7f134d61e"
-					(reference "R129")
+					(reference "R131")
 					(unit 1)
 				)
@@
 		(on_board yes)
 		(dnp no)
-		(property "Reference" "R120"
+		(property "Reference" "R122"
 			(at 176.53 59.6901 90)
 			(effects
@@
 			(project "SBC"
 				(path "/21bb932a-ec67-4661-9215-0551f718d1c0/df814d64-f889-41f0-8f1a-74d7f134d61e"
-					(reference "R120")
+					(reference "R122")
 					(unit 1)
 				)
@@
 		(on_board yes)
 		(dnp no)
-		(property "Reference" "R139"
+		(property "Reference" "R141"
 			(at 40.64 182.8801 90)
 			(effects
@@
 			(project "SBC"
 				(path "/21bb932a-ec67-4661-9215-0551f718d1c0/df814d64-f889-41f0-8f1a-74d7f134d61e"
-					(reference "R139")
+					(reference "R141")
 					(unit 1)
 				)
@@
 		(on_board yes)
 		(dnp no)
-		(property "Reference" "R119"
+		(property "Reference" "R121"
 			(at 166.37 59.6901 90)
 			(effects
@@
 			(project "SBC"
 				(path "/21bb932a-ec67-4661-9215-0551f718d1c0/df814d64-f889-41f0-8f1a-74d7f134d61e"
-					(reference "R119")
+					(reference "R121")
 					(unit 1)
 				)
@@
 		(on_board yes)
 		(dnp yes)
-		(property "Reference" "R133"
+		(property "Reference" "R135"
 			(at 40.64 162.5601 90)
 			(effects
@@
 			(project "SBC"
 				(path "/21bb932a-ec67-4661-9215-0551f718d1c0/df814d64-f889-41f0-8f1a-74d7f134d61e"
-					(reference "R133")
+					(reference "R135")
 					(unit 1)
 				)
@@
 		(on_board yes)
 		(dnp yes)
-		(property "Reference" "R138"
+		(property "Reference" "R140"
 			(at 120.6501 171.45 90)
 			(effects
@@
 			(project "SBC"
 				(path "/21bb932a-ec67-4661-9215-0551f718d1c0/df814d64-f889-41f0-8f1a-74d7f134d61e"
-					(reference "R138")
+					(reference "R140")
 					(unit 1)
 				)
@@
 		(on_board yes)
 		(dnp no)
-		(property "Reference" "R121"
+		(property "Reference" "R123"
 			(at 186.69 59.6901 90)
 			(effects
@@
 			(project "SBC"
 				(path "/21bb932a-ec67-4661-9215-0551f718d1c0/df814d64-f889-41f0-8f1a-74d7f134d61e"
-					(reference "R121")
+					(reference "R123")
 					(unit 1)
 				)
@@
 		(on_board yes)
 		(dnp yes)
-		(property "Reference" "R137"
+		(property "Reference" "R139"
 			(at 107.95 163.8301 90)
 			(effects
@@
 			(project "SBC"
 				(path "/21bb932a-ec67-4661-9215-0551f718d1c0/df814d64-f889-41f0-8f1a-74d7f134d61e"
-					(reference "R137")
+					(reference "R139")
 					(unit 1)
 				)
@@
 		(on_board yes)
 		(dnp yes)
-		(property "Reference" "R132"
+		(property "Reference" "R134"
 			(at 187.96 148.5901 90)
 			(effects
@@
 			(project "SBC"
 				(path "/21bb932a-ec67-4661-9215-0551f718d1c0/df814d64-f889-41f0-8f1a-74d7f134d61e"
-					(reference "R132")
+					(reference "R134")
 					(unit 1)
 				)
@@
 		(on_board yes)
 		(dnp yes)
-		(property "Reference" "R130"
+		(property "Reference" "R132"
 			(at 163.83 148.5901 90)
 			(effects
@@
 			(project "SBC"
 				(path "/21bb932a-ec67-4661-9215-0551f718d1c0/df814d64-f889-41f0-8f1a-74d7f134d61e"
-					(reference "R130")
+					(reference "R132")
 					(unit 1)
 				)
@@
 		(on_board yes)
 		(dnp no)
-		(property "Reference" "R131"
+		(property "Reference" "R133"
 			(at 177.8 148.5901 90)
 			(effects
@@
 			(project "SBC"
 				(path "/21bb932a-ec67-4661-9215-0551f718d1c0/df814d64-f889-41f0-8f1a-74d7f134d61e"
-					(reference "R131")
+					(reference "R133")
 					(unit 1)
 				)
@@
 		(on_board yes)
 		(dnp no)
-		(property "Reference" "R136"
+		(property "Reference" "R138"
 			(at 74.93 162.5601 90)
 			(effects
@@
 			(project "SBC"
 				(path "/21bb932a-ec67-4661-9215-0551f718d1c0/df814d64-f889-41f0-8f1a-74d7f134d61e"
-					(reference "R136")
+					(reference "R138")
 					(unit 1)
 				)
@@
 		(on_board yes)
 		(dnp no)
-		(property "Reference" "R124"
+		(property "Reference" "R126"
 			(at 139.6999 93.98 90)
 			(effects
@@
 			(project "SBC"
 				(path "/21bb932a-ec67-4661-9215-0551f718d1c0/df814d64-f889-41f0-8f1a-74d7f134d61e"
-					(reference "R124")
+					(reference "R126")
 					(unit 1)
 				)
@@
 		(on_board yes)
 		(dnp yes)
-		(property "Reference" "R140"
+		(property "Reference" "R142"
 			(at 52.07 182.8801 90)
 			(effects
@@
 			(project "SBC"
 				(path "/21bb932a-ec67-4661-9215-0551f718d1c0/df814d64-f889-41f0-8f1a-74d7f134d61e"
-					(reference "R140")
+					(reference "R142")
 					(unit 1)
 				)
@@
 		(on_board yes)
 		(dnp yes)
-		(property "Reference" "R127"
+		(property "Reference" "R129"
 			(at 77.47 116.8399 90)
 			(effects
@@
 			(project "SBC"
 				(path "/21bb932a-ec67-4661-9215-0551f718d1c0/df814d64-f889-41f0-8f1a-74d7f134d61e"
-					(reference "R127")
+					(reference "R129")
 					(unit 1)
 				)
@@
 		(on_board yes)
 		(dnp no)
-		(property "Reference" "R128"
+		(property "Reference" "R130"
 			(at 271.78 132.0799 90)
 			(effects
@@
 			(project "SBC"
 				(path "/21bb932a-ec67-4661-9215-0551f718d1c0/df814d64-f889-41f0-8f1a-74d7f134d61e"
-					(reference "R128")
+					(reference "R130")
 					(unit 1)
 				)
@@
 		(on_board yes)
 		(dnp no)
-		(property "Reference" "R118"
+		(property "Reference" "R120"
 			(at 156.21 59.6901 90)
 			(effects
@@
 			(project "SBC"
 				(path "/21bb932a-ec67-4661-9215-0551f718d1c0/df814d64-f889-41f0-8f1a-74d7f134d61e"
-					(reference "R118")
+					(reference "R120")
 					(unit 1)
 				)

Commit message: More routing
Changed lines of the file:
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@@
 			)
 		)
-		(property "Description" "MLCC"
+		(property "Description" ""
 			(at 282.194 41.91 0)
 			(effects
@@
 		(exclude_from_sim no)
 		(in_bom yes)
-		(on_board yes)
+		(on_board no)
 		(dnp yes)
 		(property "Reference" "C71"
@@
 		(exclude_from_sim no)
 		(in_bom yes)
-		(on_board yes)
+		(on_board no)
 		(dnp yes)
 		(property "Reference" "C72"
@@
 		(exclude_from_sim no)
 		(in_bom yes)
-		(on_board yes)
+		(on_board no)
 		(dnp yes)
 		(property "Reference" "C69"
@@
 		(exclude_from_sim no)
 		(in_bom yes)
-		(on_board yes)
+		(on_board no)
 		(dnp yes)
 		(property "Reference" "C70"
