File: mpu.kicad_sch (KiCad schematic)
At the start: 97 parts, among them J1 USB_OTG, J2 Conn_ARM_JTAG_SWD_20, J3 USB_OTG, J4 Conn_02x20_Counter_Clockwise, U3 ECMF02-2AMX6, U4 ECMF02-2AMX6, U9 STM32MP153AABx, X1 ASE-24MHz

Commit message: Started an entire reroute
Parts:
- removed J4: Conn_02x20_Counter_Clockwise, Connector_PinHeader_1.27mm:PinHeader_2x20_P1.27mm_Vertical, symbol Connector_Generic:Conn_02x20_Counter_Clockwise
- added J4: Conn_02x25_Counter_Clockwise, Connector_PinHeader_2.54mm:PinHeader_2x25_P2.54mm_Vertical, symbol Connector_Generic:Conn_02x25_Counter_Clockwise
- D15, D16: footprint SparkFun-LED:LED_0603_1608Metric -> LED_SMD:LED_0603_1608Metric
- JP1, JP2, JP3: footprint SparkFun-Jumper:Jumper_2_NO -> Jumper:SolderJumper-2_P1.3mm_Open_Pad1.0x1.5mm
- SW1: footprint SparkFun-Switch:Push_SMD_4.2x3.2mm -> Button_Switch_SMD:SW_Push_1P1T_NO_CK_KSC6xxG
- TP20, TP21: footprint SparkFun-Connector:TestPoint-0.5mm -> TestPoint:TestPoint_Pad_1.0x1.0mm

Commit message: Routing Power
Parts:
- added C102, C103, C104: 1uF, Capacitor_SMD:C_0201_0603Metric, symbol SparkFun-Capacitor:C
Connections:
- net GND: now also C102.2, C103.2, C104.2
- net VDD: now also C103.1, C104.1
- net VDD_CORE: now also C102.1

Commit message: Routing ethernet
Parts:
- removed C42, C43, C44: 1uF, Capacitor_SMD:C_0402_1005Metric, symbol SparkFun-Capacitor:C
- removed C45: 1uF, Capacitor_SMD:C_0201_0603Metric, symbol SparkFun-Capacitor:C
- added J5: Conn_01x06_Pin, Connector_PinSocket_2.54mm:PinSocket_1x06_P2.54mm_Vertical, symbol Connector:Conn_01x06_Pin
Connections:
- net GND: now also J5.1 (Pin_1)
- net JTCK: now also CR3.4 (I/O); no longer CR3.5 (I/O)
- net JTMS: now also CR3.5 (I/O); no longer CR3.4 (I/O)
- net UART4_CTS: now also J5.6 (Pin_6)
- net UART4_RTS: now also J5.2 (Pin_2)
- net UART4_RX: now also CR8.3 (I/O), J5.4 (Pin_4); no longer CR8.1 (I/O)
- net UART4_TX: now also CR8.1 (I/O), J5.5 (Pin_5); no longer CR8.3 (I/O)
- net VDD: now also J5.3 (Pin_3)

Commit message: Routing Eth
Parts:
- removed C47, C48: 2.2uF, Capacitor_SMD:C_0402_1005Metric, symbol SparkFun-Capacitor:C
- removed R31: 22, Resistor_SMD:R_0402_1005Metric, symbol SparkFun-Resistor:R
Connections:
- net ETH_CLK_R: no longer names the net of U9.U7 (PG8)
- net VDD1V8_DSI renamed VDDA1V8_REG
Other:
- moved on the sheet: C53, C56

Commit message: Routed UART4 and OSC
Parts:
- removed JP1, JP2, JP3: SolderJumper_2_Open, Jumper:SolderJumper-2_P1.3mm_Open_Pad1.0x1.5mm, symbol Jumper:SolderJumper_2_Open
- added R83, R84, R85: 0, Resistor_SMD:R_0402_1005Metric, symbol SparkFun-Resistor:R
Connections:
- net BOOT0: now also R83.1
- net BOOT1: now also R84.1
- net BOOT2: now also R85.1
- net UART4_RX: now also U9.B10 (PD2); no longer U9.W6 (PB8)
- net UART4_TX: now also U9.C11 (PC8); no longer U9.T13 (PB2)
- net at R28.2: now also R83.2
- net at R29.2: now also R84.2
- net at R30.2: now also R85.2

Commit message: Routing power and fixing minor things
Connections:
- net ETH_PHY_INTn: no longer names the net of U9.F1 (PG12)
Other:
- moved on the sheet: C49, C50, C51, C52, C53, C55, C56, C57, C58

Commit message: Cleaning up routing
Parts:
- TP20, TP21: footprint TestPoint:TestPoint_Pad_1.0x1.0mm -> SparkFun-Connector:TestPoint-0.5mm
Changed lines of the file:
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@@
 			)
 		)
-		(property "Footprint" "TestPoint:TestPoint_Pad_1.0x1.0mm"
+		(property "Footprint" "SparkFun-Connector:TestPoint-0.5mm"
 			(at 742.95 208.28 0)
 			(effects
@@
 			)
 		)
-		(property "Footprint" "TestPoint:TestPoint_Pad_1.0x1.0mm"
+		(property "Footprint" "SparkFun-Connector:TestPoint-0.5mm"
 			(at 740.41 203.2 0)
 			(effects

Commit message: Finished main routing
Parts:
- SW1: footprint Button_Switch_SMD:SW_Push_1P1T_NO_CK_KSC6xxG -> Button_Switch_SMD:SW_Push_1P1T_NO_CK_KSC6xxJ
Other:
- moved on the sheet: C10, C102, C103, C104, C11, C12, C13, C14, C15, C16, C17, C18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
