File: Power.kicad_sch (KiCad schematic)
At the start: 90 parts, among them U1 STPMIC1APQR

Commit message: Cleaning up routing
Parts:
- TP1, TP10, TP11, TP12, TP13, TP14, TP15, TP16, TP2, TP3, TP4, TP5, TP6, TP7, TP8, TP9: footprint TestPoint:TestPoint_Pad_1.0x1.0mm -> SparkFun-Connector:TestPoint-0.5mm
Changed lines of the file:
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@@
 			)
 		)
-		(property "Footprint" "TestPoint:TestPoint_Pad_1.0x1.0mm"
+		(property "Footprint" "SparkFun-Connector:TestPoint-0.5mm"
 			(at 80.01 134.62 0)
 			(effects
@@
 			)
 		)
-		(property "Footprint" "TestPoint:TestPoint_Pad_1.0x1.0mm"
+		(property "Footprint" "SparkFun-Connector:TestPoint-0.5mm"
 			(at 172.72 113.03 0)
 			(effects
@@
 			)
 		)
-		(property "Footprint" "TestPoint:TestPoint_Pad_1.0x1.0mm"
+		(property "Footprint" "SparkFun-Connector:TestPoint-0.5mm"
 			(at 151.13 140.97 0)
 			(effects
@@
 			)
 		)
-		(property "Footprint" "TestPoint:TestPoint_Pad_1.0x1.0mm"
+		(property "Footprint" "SparkFun-Connector:TestPoint-0.5mm"
 			(at 38.1 156.21 0)
 			(effects
@@
 			)
 		)
-		(property "Footprint" "TestPoint:TestPoint_Pad_1.0x1.0mm"
+		(property "Footprint" "SparkFun-Connector:TestPoint-0.5mm"
 			(at 198.12 113.03 0)
 			(effects
@@
 			)
 		)
-		(property "Footprint" "TestPoint:TestPoint_Pad_1.0x1.0mm"
+		(property "Footprint" "SparkFun-Connector:TestPoint-0.5mm"
 			(at 222.25 140.97 0)
 			(effects
@@
 			)
 		)
-		(property "Footprint" "TestPoint:TestPoint_Pad_1.0x1.0mm"
+		(property "Footprint" "SparkFun-Connector:TestPoint-0.5mm"
 			(at 267.97 140.97 0)
 			(effects
@@
 			)
 		)
-		(property "Footprint" "TestPoint:TestPoint_Pad_1.0x1.0mm"
+		(property "Footprint" "SparkFun-Connector:TestPoint-0.5mm"
 			(at 100.33 173.99 0)
 			(effects
@@
 			)
 		)
-		(property "Footprint" "TestPoint:TestPoint_Pad_1.0x1.0mm"
+		(property "Footprint" "SparkFun-Connector:TestPoint-0.5mm"
 			(at 100.33 156.21 0)
 			(effects
@@
 			)
 		)
-		(property "Footprint" "TestPoint:TestPoint_Pad_1.0x1.0mm"
+		(property "Footprint" "SparkFun-Connector:TestPoint-0.5mm"
 			(at 38.1 175.26 0)
 			(effects
@@
 			)
 		)
-		(property "Footprint" "TestPoint:TestPoint_Pad_1.0x1.0mm"
+		(property "Footprint" "SparkFun-Connector:TestPoint-0.5mm"
 			(at 267.97 113.03 0)
 			(effects
@@
 			)
 		)
-		(property "Footprint" "TestPoint:TestPoint_Pad_1.0x1.0mm"
+		(property "Footprint" "SparkFun-Connector:TestPoint-0.5mm"
 			(at 151.13 113.03 0)
 			(effects
@@
 			)
 		)
-		(property "Footprint" "TestPoint:TestPoint_Pad_1.0x1.0mm"
+		(property "Footprint" "SparkFun-Connector:TestPoint-0.5mm"
 			(at 222.25 113.03 0)
 			(effects
@@
 			)
 		)
-		(property "Footprint" "TestPoint:TestPoint_Pad_1.0x1.0mm"
+		(property "Footprint" "SparkFun-Connector:TestPoint-0.5mm"
 			(at 172.72 140.97 0)
 			(effects
@@
 			)
 		)
-		(property "Footprint" "TestPoint:TestPoint_Pad_1.0x1.0mm"
+		(property "Footprint" "SparkFun-Connector:TestPoint-0.5mm"
 			(at 245.11 113.03 0)
 			(effects
@@
 			)
 		)
-		(property "Footprint" "TestPoint:TestPoint_Pad_1.0x1.0mm"
+		(property "Footprint" "SparkFun-Connector:TestPoint-0.5mm"
 			(at 245.11 140.97 0)
 			(effects

Commit message: Organizing REFDES
Parts:
- renumbered CVLXBST1 to C1, C94 to C10, C101 to C11, CBUCK1IN1 to C12, CBUCK2IN1 to C13, CSWOUT1 to C14, C95 to C15, C96 to C16, CLDO1OUT1 to C17, CLDO4OUT1 to C18, CBUCK3IN1 to C19, CVOUT1 to C2, CBUCK4IN1 to C20, C97 to C21, C98 to C22, CLDO2OUT1 to C23, CLDO5OUT1 to C24, CVIN1 to C25, CLDO16IN1 to C26, C100 to C27, C99 to C28, CLDO3OUT1 to C29, CVOUT3 to C3, CLDO6OUT1 to C30, CLDO3IN1 to C31, CLDO25IN1 to C32, CVOUT2 to C4, CVOUT4 to C5, CBSTOUT1 to C6, CINTLDO1 to C7, CVBUSOTG1 to C8, CVREF1 to C9, D12 to D1, D4 to D10, D9 to D11, D5 to D12, D10 to D13, D11 to D14, D1 to D2, D6 to D3, D13 to D4, D2 to D5, D7 to D6, D14 to D7, D3 to D8, D8 to D9, H3 to H2, H2 to H3, LX3 to LX2, LX2 to LX3, R14 to R1, R4 to R10, R9 to R11, R5 to R12, R10 to R13, R11 to R14, R12 to R15, R13 to R16, R1 to R2, R6 to R3, R15 to R4, R2 to R5, R7 to R6, R16 to R7, R3 to R8, R8 to R9, TP13 to TP1, TP2 to TP10, TP9 to TP11, TP3 to TP12, TP4 to TP13, TP10 to TP14, TP5 to TP15, TP11 to TP16, TP6 to TP17, TP12 to TP18, TP16 to TP2, TP7 to TP3, TP14 to TP4, TP15 to TP5, TP1 to TP6, TP8 to TP7, TP22 to TP8, TP23 to TP9
